File: pcb/LNA_V2/LNA copy.sch (EAGLE design)
At the start: 12 parts, among them X1 SMA-142-0701-801/806, X2 SMA-142-0701-801/806

Commit message: Update of pcb images.
Other:
- note added: "1/1"
- note added: "2.0.1"
- moved on the sheet: C1, C2, C3, C4, C5, D1, L1, L2, X1, X2
